File: PCB & Schematic/Slave.sch (EAGLE design)
At the start: 55 parts, among them J1 CH1, J10 CH10, J11 GND, J2 CH2, J3 CH3, J4 CH4, J5 CH5, J6 CH6, J7 CH7, J8 CH8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

Commit message: Added initial PCB layout using Eagle.
It passes design rule checks, but I should still go over
it once more by hand to sanity check everything.
Parts:
- T1, T10, T2, T3, T4, T5, T6, T7, T8, T9: device transistor-neu-to92:-NPN-TO220 -> transistor-neu-to92:-NPN-TO220V
Connections:
- net N$1 renamed HS1
- net N$11 renamed HS6
- net N$13 renamed HS7
- net N$15 renamed HS8
- net N$17 renamed HS9
- net N$2 renamed HS10
- net N$3 renamed HS2
- net N$5 renamed HS3
- net N$7 renamed HS4
- net N$9 renamed HS5
- net FEEDBACK1: now also U$1.A12; no longer U$1.14/A0
- net FEEDBACK10: now also U$1.30/A19/SDA1; no longer U$1.31/A20
- net FEEDBACK2: now also U$1.26/A15; no longer U$1.15/A1/T
- net FEEDBACK3: now also U$1.27/A16; no longer U$1.16/A2/T
- net FEEDBACK4: now also U$1.28/A17; no longer U$1.17/A3/T
- net FEEDBACK5: now also U$1.A14/DAC; no longer U$1.26/A15
- net FEEDBACK6: now also U$1.14/A0; no longer U$1.27/A16
- net FEEDBACK7: now also U$1.15/A1/T; no longer U$1.28/A17
- net FEEDBACK8: now also U$1.16/A2/T; no longer U$1.29/A18/SCL1
- net FEEDBACK9: now also U$1.17/A3/T; no longer U$1.30/A19/SDA1
